File: boards/marquee/marqee_attiny85/marqee_attiny85_new.sch (EAGLE design)
At the start: 11 parts, among them U1 ATTINY85-20PU

Commit message: class 3 materials; adds Arrow-NeoPixel PCB
Parts:
- removed CN1, CN2, CN3: (no value), adafruit-2014:JST_2PIN-THM
- removed JP1: (no value), pinhead:PINHD-1X3
- added JP2, JP3, JP4, SENSOR_INPUT: (no value), pinhead:PINHD-1X2
- added R4: 1k, resistor:R-US_0207/10
- added TIP120: (no value), pinhead:PINHD-1X3
- C2, C3: value (none) -> 47uF
- R1: value (none) -> 10k
- R2: value (none) -> 1k
- R3: value (none) -> 220
Connections:
- removed net N$6: CN2.1, JP1.2
- new net ANALOG_SENSOR_IN: R4.1, SENSOR_INPUT.1, U1.PB2_(SCK/USCK/SCL/ADC1/T0/INT0/PCINT2)
- new net THING: JP2.1, TIP120.2
- net GND: now also JP3.1, JP4.1, R4.2, TIP120.3; no longer CN1.1, CN3.1, JP1.3
- net N$2: now also TIP120.1; no longer JP1.1
- net VCC: now also JP2.2, JP3.2, JP4.2, SENSOR_INPUT.2; no longer CN1.2, CN2.2, CN3.2
Other:
- note added: "+/- Pin for LED Board"
- note added: "47uF Capacitors act like shock-absorbers"
- note added: "Base (control pin) Collector (LED ground) Emittor (PCB ground)"
- note added: "Here is a very different Looking ATtiny85 Schematic Symbol"
- note added: "LED connected to Power Very useful for debugging"
- note added: "My Analog Sensor Connects Here"
- note added: "Power input and output "Daisy-Chaining""
- note added: "Pull-Up Resistor on RESET Pin"
- note added: "TIP120 Transistor needs a 3-pin header"
- moved on the sheet: LED1, R2, R3
