File: boards/marquee-neopixel/marquee-neopixel.brd (EAGLE design)
At the start: 109 x 61 mm, 86 parts, among them U1 ATTINY85-20SU

Commit message: adds example boards for common circuits
Parts:
- R1: value (none) -> 100
- R2: value (none) -> 10k
Changed lines of the file:
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@@
 <?xml version="1.0" encoding="utf-8"?>
 <!DOCTYPE eagle SYSTEM "eagle.dtd">
-<eagle version="8.5.2">
+<eagle version="8.6.1">
 <drawing>
 <settings>
@@
 <attribute name="SPICEPREFIX" value="C" x="14.9" y="16.9" size="1.778" layer="27" rot="R180" display="off"/>
 </element>
-<element name="R1" library="eagle-ltspice" library_urn="urn:adsk.eagle:library:217" package="R0603" package3d_urn="urn:adsk.eagle:package:13302/1" value="" x="7" y="44" rot="R90">
+<element name="R1" library="eagle-ltspice" library_urn="urn:adsk.eagle:library:217" package="R0603" package3d_urn="urn:adsk.eagle:package:13302/1" value="100" x="7" y="44" rot="R90">
 <attribute name="SPICEMODEL" value="NONE" x="7" y="44" size="1.778" layer="27" rot="R90" display="off"/>
 <attribute name="SPICEPREFIX" value="R" x="7" y="44" size="1.778" layer="27" rot="R90" display="off"/>
@@
 <attribute name="SPICEPREFIX" value="C" x="11.6" y="8.9" size="1.778" layer="27" rot="R180" display="off"/>
 </element>
-<element name="R2" library="eagle-ltspice" library_urn="urn:adsk.eagle:library:217" package="R0603" package3d_urn="urn:adsk.eagle:package:13302/1" value="" x="19.3" y="15.5" rot="R180">
+<element name="R2" library="eagle-ltspice" library_urn="urn:adsk.eagle:library:217" package="R0603" package3d_urn="urn:adsk.eagle:package:13302/1" value="10k" x="19.3" y="15.5" rot="R180">
 <attribute name="SPICEMODEL" value="NONE" x="19.3" y="15.5" size="1.778" layer="27" rot="R180" display="off"/>
 <attribute name="SPICEPREFIX" value="R" x="19.3" y="15.5" size="1.778" layer="27" rot="R180" display="off"/>
