File: boards/Common_Circuits/1_Passive_Components/4-RC_Filter/Pull_Up:Down_Resistors.sch (EAGLE design)
At the start: 22 parts, among them SW1 SPST_TACT-KMR2, SW2 SPST_TACT-KMR2, SW3 SPST_TACT-KMR2

Commit message: adds ESP8266 board to common circuits
Other:
- note added: "Low-frequency "waves" are removed with HIGH-PASS FILTERS"
Changed lines of the file:
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@@
 <?xml version="1.0" encoding="utf-8"?>
 <!DOCTYPE eagle SYSTEM "eagle.dtd">
-<eagle version="8.6.1">
+<eagle version="8.6.0">
 <drawing>
 <settings>
@@
 <text x="20.32" y="91.44" size="5.08" layer="94">Data Line Filters</text>
 <text x="106.68" y="91.44" size="5.08" layer="94">High-Pass Filter</text>
-<text x="116.84" y="71.12" size="1.778" layer="91">High-frequency "spikes" are
-removed with LOW-PASS FILTERS</text>
+<text x="116.84" y="71.12" size="1.778" layer="91">Low-frequency "waves" are
+removed with HIGH-PASS FILTERS</text>
 <circle x="152.4" y="43.18" radius="12.7" width="0.1016" layer="94"/>
 <text x="106.68" y="83.82" size="1.778" layer="94">RC High-Pass Filter Calculator:
